File: AskSinPP_DinRailBoard/HM-ES-TX-WM_IEC_v1p0.brd (EAGLE design)
At the start: 33 x 86.5 mm, 30 parts, among them IC2 MCP1700T-5002E_TT, IC3 MEGA8-AI, J1 CTB0502_6, J2 CTB0502_6, M1 I2C_BREAKOUT_4P, Q1 CSTCE, U1 CC1101SMD

Commit message: LDO part number corrected
Parts:
- IC2: value MCP1700T-5002E_TT -> MCP1700T-3302E_TT
Changed lines of the file:
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@@
 <attribute name="VALUE" x="6.35" y="13.335" size="1.27" layer="27" align="center"/>
 </element>
-<element name="IC2" library="SamacSys_Parts" package="SOT95P237X112-3N" value="MCP1700T-5002E_TT" x="4.445" y="17.78" smashed="yes" rot="R270">
+<element name="IC2" library="SamacSys_Parts" package="SOT95P237X112-3N" value="MCP1700T-3302E_TT" x="4.445" y="17.78" smashed="yes" rot="R270">
 <attribute name="ARROW_PART_NUMBER" value="MCP1700T-5002E/TT" x="4.445" y="17.78" size="1.778" layer="27" rot="R270" display="off"/>
 <attribute name="ARROW_PRICE-STOCK" value="https://www.arrow.com/en/products/mcp1700t-5002ett/microchip-technology?region=nac" x="4.445" y="17.78" size="1.778" layer="27" rot="R270" display="off"/>
